File: ODB/Kicad/ODB2/ODB2.kicad_sch (KiCad schematic)
At the start: 1 part, among them U1 STM32F479ZGTx

Commit message: add boot selector + coupling + external oscillator +
Parts:
- added Boot_JP1: SolderJumper_2_Open, symbol Jumper:SolderJumper_2_Open
- added Boot_R1: 1k5, symbol Device:R
- added Boot_R2: 10k, symbol Device:R
- added Coupling_FB1: 120R, symbol Device:FerriteBead
- added Crystal_C1, Crystal_C2: 28pF, symbol Device:C
- added Crystal_R1: 20R, symbol Device:R
- added Crystal_Y1: 100MHz, symbol Device:Crystal_GND23
- added Decouple_C1, Decouple_C6: 10uF, symbol Device:C
- added Decouple_C2, Decouple_C3, Decouple_C4, Decouple_C5: 100nF, symbol Device:C
- added Decouple_C7, Decouple_C8: 10nF, symbol Device:C
- added H1, H2, H3, H4: MountingHole, symbol Mechanical:MountingHole
Connections:
- net BOOT0: now reaches U1.137 (BOOT0)
- net BOOT0: now also Boot_R1.2, Boot_R2.1
- net PH0: now reaches U1.18 (PH0)
- net PH0: now also U1.19 (PH1), Crystal_C1.1, Crystal_Y1.1
- new net: Boot_JP1.2 (B), Boot_R1.1
- new net +3.3VA: Coupling_FB1.1, Decouple_C6.1, Decouple_C7.1
- new net +3V3: Boot_JP1.1 (A), Coupling_FB1.2, Decouple_C1.1, Decouple_C2.1, Decouple_C3.1, Decouple_C4.1, Decouple_C5.1, Decouple_C8.1
- new net GND: Boot_R2.2, Crystal_C1.2, Crystal_C2.1, Crystal_C2.2, Crystal_R1.2, Crystal_Y1.2, Crystal_Y1.3, Crystal_Y1.4, Decouple_C1.2, Decouple_C2.2, Decouple_C3.2, Decouple_C4.2, Decouple_C5.2, Decouple_C6.2, Decouple_C7.2, Decouple_C8.2
- new net PH1: Crystal_R1.1
Other:
- removed sheet Pyro_Multiplex
- added sheet Pyro (Pyro.kicad_sch)
- note added: "Boot Option"
- note added: "C = 2(Cfabricant - Ctrace) = 2(18pF - 4pF) = 28pF *Ctrace ~2-5pF"
- note added: "Decoupling Capacitor"
- note added: "External Crystal"
- note added: "Mounting Hole"
- note added: "OSC_IN"
- note added: "OSC_OUT"

Commit message: add NRST
Parts:
- added RST_C1: 100nF, symbol Device:C
- added RST_R1: 10k, symbol Device:R
Connections:
- net +3V3: now also RST_R1.1
- net GND: now also RST_C1.2
- net NRST: now reaches U1.20 (NRST)
- net NRST: now also RST_C1.1, RST_R1.2
Other:
- note added: "Ajouter un bouton poussoir pour forcer un RST?"
- note added: "Vérifier res filtre (0-20R) -> 100MHz crystal"
- moved on the sheet: Coupling_FB1, Crystal_C1, Crystal_C2, Crystal_R1, Crystal_Y1, Decouple_C6, Decouple_C7, Decouple_C8

Commit message: add SWDebug connector
Connections:
- net SYS-SWDIO: now reaches U1.107 (PA13)
- net SYS_SWCLK: now reaches U1.111 (PA14)
- net VDD: now reaches U1.142 (PDR_ON)
- net SYS_SWO: now reaches U1.43 (PB2)
Other:
- note added: "C=2(Cfabricant-Ctrace)=2(18pF-4pF)=28pF *Ctrace ~2-5pF"
- note removed: "C = 2(Cfabricant - Ctrace) = 2(18pF - 4pF) = 28pF *Ctrace ~2-5pF"
- moved on the sheet: Boot_JP1, Boot_R1, Boot_R2, Coupling_FB1, Crystal_C1, Crystal_C2, Crystal_R1, Crystal_Y1, Decouple_C1, Decouple_C2, Decouple_C3, Decouple_C4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
