File: ODB/Kicad/ODB2/Pyro.kicad_sch (KiCad schematic)
At the start: 0 parts

Commit message: add SWDebug connector
Other:
- note added: "Pyros"
- company: (none) -> GAUL
- title: (none) -> Pyros
Changed lines of the file:
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@@
 	(generator_version "8.0")
 	(paper "A4")
+	(title_block
+		(title "Pyros")
+		(date "2024-11-09")
+		(company "GAUL")
+	)
+	(text "Pyros"
+		(exclude_from_sim no)
+		(at 21.59 16.51 0)
+		(effects
+			(font
+				(size 4 4)
+				(thickness 0.8)
+				(bold yes)
+			)
+		)
+	)
 )
