File: ODB/Kicad/ODB2/Sensors.kicad_sch (KiCad schematic)
At the start: 0 parts

Commit message: add SWDebug connector
Other:
- company: (none) -> GAUL
- title: (none) -> Sensors
Changed lines of the file:
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@@
 	(generator_version "8.0")
 	(paper "A4")
+	(title_block
+		(title "Sensors")
+		(date "2024-11-09")
+		(company "GAUL")
+	)
 	(text "Sensors"
 		(exclude_from_sim no)
