File: Kicad/ODB2/RFD900x.kicad_sch (KiCad schematic)
At the start: 0 parts

Commit message: edit titles
Other:
- company: (none) -> GAUL
- title: (none) -> Radio
Changed lines of the file:
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@@
 	(generator_version "8.0")
 	(paper "A4")
+	(title_block
+		(title "Radio")
+		(date "2024-11-09")
+		(company "GAUL")
+	)
 )

Commit message: add titles
Other:
- note added: "Radio"
Changed lines of the file:
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@@
 		(company "GAUL")
 	)
+	(text "Radio"
+		(exclude_from_sim no)
+		(at 26.924 18.796 0)
+		(effects
+			(font
+				(size 6 6)
+				(thickness 1.2)
+				(bold yes)
+			)
+		)
+	)
 )
