File: Kicad/ODB2/IO_Peripherals.kicad_sch (KiCad schematic)
At the start: 23 parts, among them J1 USB_B_Micro, J5 RFM_Conn_Coaxial, U10 W25Q512JVEIQ, U4 USBLC6-2P6, U9 RFM23BP-433-S2

Commit message: footprint
Parts:
- BUZ_R2, LED_R1: footprint (none) -> Resistor_SMD:R_0805_2012Metric
- BUZ_R3: value 1k5R -> 1k5; footprint (none) -> Resistor_SMD:R_0805_2012Metric
- Beacon_C1, MEM_C1: footprint (none) -> Capacitor_SMD:C_0805_2012Metric
- D3: footprint (none) -> Diode_SMD:D_SOD-123
- IO_LED1: footprint (none) -> LED_SMD:LED_0805_2012Metric
- J5: footprint (none) -> Connector_Coaxial:SMA_Wurth_60312002114503_Vertical
- LS1: footprint SMTB-0927-TW-R_PUI -> ODB:SMTB-0927-TW-R_PUI
Changed lines of the file:
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@@
 			)
 		)
-		(property "Footprint" ""
+		(property "Footprint" "LED_SMD:LED_0805_2012Metric"
 			(at 143.51 97.79 0)
 			(effects
@@
 		(on_board yes)
 		(dnp no)
-		(property "Reference" "#PWR038"
+		(property "Reference" "#PWR0105"
 			(at 17.78 71.12 0)
 			(effects
@@
 			(project "ODB2"
 				(path "/4b06c5d1-aa8b-48ed-8972-b43a60cfab78/93865dc8-71fa-4dc6-90ce-f5a9779dfd41"
-					(reference "#PWR038")
+					(reference "#PWR0105")
 					(unit 1)
 				)
@@
 		(on_board yes)
 		(dnp no)
-		(property "Reference" "#PWR037"
+		(property "Reference" "#PWR0106"
 			(at 19.05 34.29 0)
 			(effects
@@
 			(project "ODB2"
 				(path "/4b06c5d1-aa8b-48ed-8972-b43a60cfab78/93865dc8-71fa-4dc6-90ce-f5a9779dfd41"
-					(reference "#PWR037")
+					(reference "#PWR0106")
 					(unit 1)
 				)
@@
 			)
 		)
-		(property "Value" "1k5R"
+		(property "Value" "1k5"
 			(at 120.65 34.29 90)
 			(effects
@@
 			)
 		)
-		(property "Footprint" ""
+		(property "Footprint" "Resistor_SMD:R_0805_2012Metric"
 			(at 120.65 35.052 90)
 			(effects
@@
 		(on_board yes)
 		(dnp no)
-		(property "Reference" "#PWR039"
+		(property "Reference" "#PWR0107"
 			(at 31.75 34.29 0)
 			(effects
@@
 			(project "ODB2"
 				(path "/4b06c5d1-aa8b-48ed-8972-b43a60cfab78/93865dc8-71fa-4dc6-90ce-f5a9779dfd41"
-					(reference "#PWR039")
+					(reference "#PWR0107")
 					(unit 1)
 				)
@@
 			)
 		)
-		(property "Footprint" ""
+		(property "Footprint" "Resistor_SMD:R_0805_2012Metric"
 			(at 133.35 96.012 90)
 			(effects
@@
 			)
 		)
-		(property "Footprint" ""
+		(property "Footprint" "Connector_Coaxial:SMA_Wurth_60312002114503_Vertical"
 			(at 259.08 134.62 0)
 			(effects
@@
 			)
 		)
-		(property "Footprint" ""
+		(property "Footprint" "Resistor_SMD:R_0805_2012Metric"
 			(at 142.24 46.482 90)
 			(effects
@@
 			)
 		)
-		(property "Footprint" ""
+		(property "Footprint" "Capacitor_SMD:C_0805_2012Metric"
 			(at 260.35 123.4948 0)
 			(effects
@@
 			)
 		)
-		(property "Footprint" "SMTB-0927-TW-R_PUI"
+		(property "Footprint" "ODB:SMTB-0927-TW-R_PUI"
 			(at 138.938 43.942 0)
 			(effects
@@
 		(dnp no)
 		(fields_autoplaced yes)
-		(property "Reference" "#PWR042"
+		(property "Reference" "#PWR0103"
 			(at 72.39 80.01 0)
 			(effects
@@
 			(project "ODB2"
 				(path "/4b06c5d1-aa8b-48ed-8972-b43a60cfab78/93865dc8-71fa-4dc6-90ce-f5a9779dfd41"
-					(reference "#PWR042")
+					(reference "#PWR0103")
 					(unit 1)
 				)
@@
 			)
 		)
-		(property "Footprint" ""
+		(property "Footprint" "Capacitor_SMD:C_0805_2012Metric"
 			(at 259.3848 96.52 0)
 			(effects
@@
 		(dnp no)
 		(fields_autoplaced yes)
-		(property "Reference" "#PWR040"
+		(property "Reference" "#PWR0104"
 			(at 31.75 57.15 0)
 			(effects
@@
 			(project "ODB2"
 				(path "/4b06c5d1-aa8b-48ed-8972-b43a60cfab78/93865dc8-71fa-4dc6-90ce-f5a9779dfd41"
-					(reference "#PWR040")
+					(reference "#PWR0104")
 					(unit 1)
 				)
@@
 			)
 		)
-		(property "Footprint" ""
+		(property "Footprint" "Diode_SMD:D_SOD-123"
 			(at 138.43 44.45 0)
 			(effects
@@
 		(on_board yes)
 		(dnp no)
-		(property "Reference" "#PWR041"
+		(property "Reference" "#PWR0108"
 			(at 72.39 54.61 0)
 			(effects
@@
 			(project "ODB2"
 				(path "/4b06c5d1-aa8b-48ed-8972-b43a60cfab78/93865dc8-71fa-4dc6-90ce-f5a9779dfd41"
-					(reference "#PWR041")
-					(unit 1)
-				)
+					(reference "#PWR0108")
+					(unit 1)
+				)

Commit message: fix and gate
Other:
- note added: "Data USB + connecté"
- moved on the sheet: BUZ_Q4, BUZ_R2, BUZ_R3, IO_LED1, LED_R1

Commit message: ajout footprints
Parts:
- U10: footprint W25Q512JVEIQ:SON127P600X800X80-9N -> Library:SON127P600X800X80-9N
Changed lines of the file:
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@@
 			)
 		)
-		(property "Footprint" "W25Q512JVEIQ:SON127P600X800X80-9N"
+		(property "Footprint" "Library:SON127P600X800X80-9N"
 			(at 236.474 118.872 0)
 			(effects
