File: ODB_V3/Hardware/Kicad/ODB2/ODB2.kicad_pcb (KiCad board)
At the start: 6 copper layers, 63.1 x 114.6 mm, 237 parts, among them IC1 W25Q512JVEIQ, J1 Screw_Terminal_01x08, J10 GPS_Conn_02x04_Top_Bottom, J11 Conn_02x04_Odd_Even, J15 Vin_XT30PW-F, J2 RFD_GT17HN-4DP-2HA56, J3 SYS_SW_Conn_01x05_Header, J5 MEM2067, J6 IdeFIX_GT17HN-4DP-2HA56, U1 STM32F412ZGTx, U10 ADXL382-2BCCZ-RL7, U11 SI5442DU-T1-GE3, U12 SI5442DU-T1-GE3, U13 L6981N33DR, U2 LM339, U3 SI5442DU-T1-GE3, U4 MS580301BA01-00, U6 BNO055, U7 MPQ9843GLE-5-AEC1-Z, U8 SI5442DU-T1-GE3, U9 MAX6612MXK, Y1 ABM8G-25.000MHZ-18-D2Y-T

Commit message: wip: tuning + remove silkscreen + add 3d models
Parts:
- moved SD_C1 43.9 mm to (174.4, 103.1)
- moved MEM_C1 18.0 mm to (128.6, 92.9), turned to 0 degrees
- moved BARO_C1 7.53 mm to (143.8, 119.9), turned to 180 degrees
- moved Crystal_R1 5.90 mm to (139.7, 93.5)
- moved Crystal_C1 4.51 mm to (142.5, 96.8), turned to 90 degrees
- moved Crystal_R2 4.14 mm to (140.0, 99.7), turned to 180 degrees
- moved Crystal_C2 3.91 mm to (137.3, 96.1), turned to -90 degrees
- moved MEM_R3 2.82 mm to (128.6, 96.0)
- moved MEM_R4 2.82 mm to (128.6, 97.6)
- moved IC1 1.91 mm to (122.2, 96.1)
- moved Y1 1.90 mm to (139.9, 96.4), turned to 180 degrees
- moved MEM_R6 1.83 mm to (128.6, 99.1)
- moved VCAP_C1 1.82 mm to (165.6, 109.6), turned to -90 degrees
- moved U4 1.66 mm to (141.9, 115.5), turned to 0 degrees
- moved IMU_C4 1.65 mm to (169.2, 60.4)
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Other:
- outline, holes or cut-outs redrawn
