File: ODB_V3/Hardware/Kicad/ODB2/_autosave-ODB2.kicad_pcb (KiCad board)
At the start: 6 copper layers, 63.1 x 114.6 mm, 248 parts, among them J1 142-0701-801, J10 MEM2067, J2 0436500404, J3 0436500404, J4 USB_B_Micro, J5 SYS_SW_Conn_01x06_Header, J7 Conn_02x04_Odd_Even, J8 Vin_XT30PW-F, J9 Screw_Terminal_01x08, Q1 MMBT3904, Q2 SI7617DN-T1-GE3, Q3 MMBT3904, Q4 SI7617DN-T1-GE3, U1 HM11, U10 SI5442DU-T1-GE3, U11 SI5442DU-T1-GE3, U12 SI5442DU-T1-GE3, U13 MS561101BA03-50, U14 L6981N33DR, U15 MPQ9843GLE-5-AEC1-Z, U16 USBLC6-2P6, U2 L76L-M33, U3 MAX6612MXK, U4 BNO055, U5 ADXL382-2BCCZ-RL7, U6 LM339B, U7 SI5442DU-T1-GE3, U8 STM32F412ZGTx, U9 W25Q512JVEIQ, Y1 ABM8G-25.000MHZ-18-D2Y-T

Commit message: modify PCB to fix all fixes except pyro injector and silkscreen
Parts:
- moved G*** 12.9 mm to (103.4, 67.4)
Changed lines of the file:
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@@
 	(footprint "ODB:Logo-QC"
 		(layer "F.Cu")
-		(at 105.855861 54.768627)
+		(at 103.423478 67.413379)
 		(property "Reference" "G***"
 			(at 0 0 0)
